File: PCBs/breakoutboard-V2.kicad_sch (KiCad schematic)
At the start: 36 parts, among them IC1 PASCO2V01BUMA1, IC2 BMP390, IC3 MT3608, J2 Conn_01x02, J3 BHR-24-VUA, J4 SM06B-GHS-TB, J5 USB_C_Receptacle, U2 ESP32-S3-WROOM-1-N16R2, U3 WS2812B-B, U4 WS2812B-B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

Commit message: Main Board PCB Updates
Main Board PCB .SCH and .PCB files.
Missing pin assignment for epaper display. Needs confirmation with Sponsor.
Parts:
- removed C2: 0.1UF-0402-16V-10%, 0402, symbol SparkFun-Capacitors:0.1UF-0402-16V-10%
- removed C3, C4: 1.0UF-0603-16V-10%, 0603, symbol SparkFun-Capacitors:1.0UF-0603-16V-10%
- removed C5, C7: 22UF-0805-6.3V-20%, 0805, symbol SparkFun-Capacitors:22UF-0805-6.3V-20%
- removed D1: D_Schottky_0.5A_40V_0.42V, SparkFun-Semiconductor-Standard:SOD-323, symbol SparkFun-DiscreteSemi:D_Schottky_0.5A_40V_0.42V
- removed IC2: BMP390, BMP390, symbol BMP390:BMP390
- removed IC3: MT3608, SOT95P280X145-6N, symbol MT3608:MT3608
- removed J2: Conn_01x02, SparkFun-Connector:1X02, symbol SparkFun-Connector:Conn_01x02
- removed J3: BHR-24-VUA, SHDR24W64P254_2X12_3808X880X910P, symbol BHR-24-VUA:BHR-24-VUA
- removed L1: INDUCTOR-CDRH-4.7UH, INDUCTOR_4.7UH, symbol SparkFun-Coils:INDUCTOR-CDRH-4.7UH
- removed R6: 2.2k, 0603, symbol SparkFun-Resistors:RESISTOR0603
- removed R7: 39k, 0603, symbol SparkFun-Resistors:RESISTOR0603
- removed R8: 2.7k, 0603, symbol SparkFun-Resistors:RESISTOR0603
- removed U3, U4: WS2812B-B, WS2812B-B:LED_WS2812B-B, symbol WS2812B-B:WS2812B-B
- removed U6: CH340C, SparkFun-Semiconductor-Standard:SO16, symbol SparkFun-IC-Comm:CH340C
- added C10: 470pF, SparkFun-Capacitor:C_0603_1608Metric, symbol SparkFun-Capacitor:470pF_0603_50V_10%
- added C11: 4.7uF, SparkFun-Capacitor:C_0603_1608Metric, symbol SparkFun-Capacitor:4.7uF_0603_35V_20%
- added C12: 47uF, SparkFun-Capacitor:PANASONIC_D, symbol SparkFun-Capacitor:47uF_35V_20%
- added C13: 0.1uF, SparkFun-Capacitor:C_0603_1608Metric, symbol SparkFun-Capacitor:0.1uF_0603_25V_20%
- added C14: 10nF, SparkFun-Capacitor:C_0603_1608Metric, symbol SparkFun-Capacitor:10nF_0603_50V_10%
- added C6: 10uF, SparkFun-Capacitor:C_0603_1608Metric, symbol SparkFun-Capacitor:10uF_0603_6.3V_20%
- added D5: 0.5A, SparkFun-Semiconductor-Standard:SOD-323, symbol SparkFun-DiscreteSemi:D_Schottky_0.5A_40V_0.42V
- added J1: Conn_01x12_FPC_0.5mm, SparkFun-Connector:FPC_12_0.5MM, symbol SparkFun-Connector:Conn_01x12_FPC_0.5mm
- added L2: 10uH, SparkFun-Capacitor:C_0805_2012Metric, symbol SparkFun-Coil:10uH_0805_0.35A
- added R13: RESISTOR0402-120 ohm, 0402, symbol SparkFun-Resistors:RESISTOR0402
- added R14: 100k, SparkFun-Resistor:R_0603_1608Metric, symbol SparkFun-Resistor:100k_0603
- added R15: 47k, SparkFun-Resistor:R_0603_1608Metric, symbol SparkFun-Resistor:47k_0603
- added R16: 5.62k, SparkFun-Resistor:R_0603_1608Metric, symbol SparkFun-Resistor:5.62k_0603
- added R7: 10k, SparkFun-Resistor:R_0402_1005Metric, symbol SparkFun-Resistor:10k_0402
- added SW1, SW2: SMD_4.6x2.8mm_h2.5mm, SparkFun-Switch:Momentary_SMD_4.6x2.8mm_h2.5mm, symbol SparkFun-Switch:SPST_Momentary_SMD_4.6x2.8mm_h2.5mm
- added SW3: PTH_RA_h7.5mm, SparkFun-Switch:Momentary_PTH_RA_8-020_h7.5mm, symbol SparkFun-Switch:SPST_Momentary_PTH_RA_h7.5mm
- added U1: AP3012, SparkFun-Semiconductor-Standard:SOT23-5, symbol SparkFun-IC-Power:AP3012
- GS1: value GAS_SENSORMQ-4 -> MQ-4
Connections:
- net RST_N is gone; now on net SCL: U2.17 (IO9)
- net 12V: now also C10.1, C11.1, C12.1, C13.1, C14.1, D5.C, R15.1
- net 3.3VOUT: now also C6.1, L2.1, R13.1, R14.1, R7.1, U1.5 (IN)
- net GND: now also C11.2, C12.2, C13.2, C14.2, C6.2, J1.8 (Pin_8), R16.2, SW1.1 (A), SW2.1 (A), SW3.1 (A), U1.2 (GND)
- net SCL: no longer U2.9 (IO16)
- net SDA: now also U2.12 (IO8); no longer U2.8 (IO15)
- net D+: now reaches J5.A6 (D+), J5.B6 (D+)
- net D+: now also U2.14 (IO20)
- net D-: now reaches J5.A7 (D-), J5.B7 (D-)
- net D-: now also U2.13 (IO19)
- net ESP_0: now reaches U2.27 (IO0)
- net ESP_0: now also R7.2, SW2.2 (B)
- net CH340-RX: no longer names the net of U2.37 (TXD0)
- net CH340-TX: no longer names the net of U2.36 (RXD0)
- net button renamed RESET
- net RESET: now also SW1.2 (B), SW3.2 (B)
- new net: D5.A, L2.2, U1.1 (SW)
- new net: C10.2, R15.2, R16.1, U1.3 (FB)
- new net: R14.2, U1.4 (~{SHDN})
- new net: J1.1 (Pin_1), R13.2
- new net BUSY_N(GPIO): J1.2 (Pin_2)
- new net CSB(SPI): J1.5 (Pin_5)
- new net D/C(GPIO): J1.6 (Pin_6)
- new net RST_N(GPIO): J1.7 (Pin_7)
- new net SCL-Epaper(SPI): J1.3 (Pin_3)
- new net SDA-Epaper(SPI): J1.4 (Pin_4)
- no-connect marks 20 -> 35
Other:
- note added: "External Reset Button"
- note added: "GPIO/BOOT BUTTON"
- note added: "RESET BUTTON"
- note removed: "3.3 V LDO"
- note removed: "LED backlight"
- note removed: "RESET"
- moved on the sheet: C1, C8, C9, D3, J4, R10, R3, U5
