File: PCBs/breakoutboard-V2.kicad_pcb (KiCad board)
At the start: 2 copper layers, 40.4 x 70 mm, 39 parts, among them IC1 PASCO2V01BUMA1, J1 Conn_01x12_FPC_0.5mm, J2 Qwiic_RA, J4 SM06B-GHS-TB, J5 USB_C_Receptacle, SW1 SMD_4.6x2.8mm_h2.5mm, SW2 SMD_4.6x2.8mm_h2.5mm, SW3 PTH_RA_h7.5mm, U1 AP3012, U2 ESP32-S3-WROOM-1-N16R2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

Commit message: Update Main Board PCB
Replaced ESP32 WROOM with ESP32 mini. READY FOR AIR WIRE REVIEW :D
Parts:
- removed the G*** at (148.5, 95.2)
- removed R7, R9: 10k, SparkFun-Resistor:R_0402_1005Metric
- removed U2: ESP32-S3-WROOM-1-N16R2, ESP32-S3-WROOM-1-N16R2:XCVR_ESP32-S3-WROOM-1-N16R2
- added G***: LOGO, SparkFun-Aesthetic:SparkFun_Logo_15mm, F.Cu at (149.1, 97.4)
- added R6: 10k, SparkFun-Resistor:R_0402_1005Metric, F.Cu at (132.6, 62.9)
- added R8: 10k, SparkFun-Resistor:R_0402_1005Metric, F.Cu at (135.5, 69.9)
- added U3: ESP32-S3-MINI, SparkFun-RF:ESP32-MINI, F.Cu at (149.7, 109.8)
- moved SW1 1.17 mm to (131.9, 58.9)
- moved SW2 1.02 mm to (131.9, 68.8)
- moved R13 0.49 mm to (137.4, 115.7)
- moved D3 0.24 mm to (135.9, 65.1)
Connections:
- C12 pad +: (no net) -> /12V
- C12 pad -: (no net) -> GND
- J1 pad 5: /CSB(SPI) -> /CSB(GPIO)
- J1 pad 6: /D/C(GPIO) -> /D/C(SPI)
