File: PCBs/EpaperDisplayPCB.kicad_pcb (KiCad board)
At the start: 2 copper layers, 84 x 40.1 mm, 21 parts, among them J1 Conn_01x08, J2 Conn_01x12_FPC_0.5mm, Q1 AO3404A, U1 ePaper-2.1

Commit message: fuck you
Parts:
- removed the J2 at (152.6, 87.5)
- added FID1: Fiducial_0.5mm, SparkFun-Aesthetic:Fiducial_0.5mm_Mask1mm, F.Cu at (122.8, 104.1)
- added FID2: Fiducial_0.5mm, SparkFun-Aesthetic:Fiducial_0.5mm_Mask1mm, F.Cu at (195.2, 72.9)
- added FID3: Fiducial_0.5mm, SparkFun-Aesthetic:Fiducial_0.5mm_Mask1mm, B.Cu at (195.2, 103.4)
- added FID4: Fiducial_0.5mm, SparkFun-Aesthetic:Fiducial_0.5mm_Mask1mm, B.Cu at (122.2, 71.0)
- added G***: LOGO, SparkFun-Aesthetic:SparkFun_Logo_NoFlame_12.5mm, F.Cu at (143.8, 100.2)
- added J1: Conn_01x12_FPC_0.5mm, SparkFun-Connector:FPC_12_0.5MM, F.Cu at (154.6, 88.2)
- added Ref**: Val**, SparkFun-Aesthetic:OSHW_Logo_6mm, F.Cu at (133.6, 100.2)
- added kibuzzard-65B1FFD4: G***, kibuzzard-65B1FFD4, F.Cu at (120.1, 78.1)
- added kibuzzard-65B1FFE5: G***, kibuzzard-65B1FFE5, F.Cu at (120.3, 80.6)
- added kibuzzard-65B20022: G***, kibuzzard-65B20022, F.Cu at (120.3, 83.1)
- added kibuzzard-65B20037: G***, kibuzzard-65B20037, F.Cu at (120.3, 85.6)
- added kibuzzard-65B20040: G***, kibuzzard-65B20040, F.Cu at (120.3, 88.2)
- added kibuzzard-65B2004E: G***, kibuzzard-65B2004E, F.Cu at (120.3, 90.7)
- added kibuzzard-65B2005D: G***, kibuzzard-65B2005D, F.Cu at (120.3, 93.3)
- added kibuzzard-65B2006B: G***, kibuzzard-65B2006B, F.Cu at (120.3, 95.8)
- added kibuzzard-65B200B7: G***, kibuzzard-65B200B7, F.Cu at (195.2, 97.1)
- added kibuzzard-65B200B7: G***, kibuzzard-65B200B7, F.Cu at (195.2, 82.5)
- added kibuzzard-65B200D7: G***, kibuzzard-65B200D7, F.Cu at (154.6, 93.3)
- added kibuzzard-65B20298: G***, kibuzzard-65B20298, F.Cu at (161.5, 74.2)
- U1: value ePaper-2.1 -> ePaper-2.66; footprint SparkFun-Display:ePaper-2.13 -> SparkFun-Display:ePaper-2.66
- renumbered J1 to J2
Connections:
- J2 pad 1: ~{RST} -> +3.3V
- J2 pad 3: ~{CS} -> ~{RST}
- J2 pad 4: SCLK -> D/~{C}
- J2 pad 5: SDIO -> ~{CS}
- J2 pad 6: D/~{C} -> SCLK
- J2 pad 7: +3.3V -> SDIO
Routing:
- net +3.3V: track 91.3 -> 100.8 mm
- net ~{RST}: track 74.4 -> 66.9 mm, vias 2 -> 0
- net ~{CS}: track 66.3 -> 64.5 mm, vias 2 -> 0
- net D/~{C}: track 66.3 -> 64.8 mm
- net Net-(Q1-D): track 59.0 -> 57.6 mm
- net GND: track 27.6 -> 26.6 mm
- net SDIO: track 65.3 -> 66.2 mm, vias 2 -> 0
- net SCLK: track 66.0 -> 65.4 mm, vias 2 -> 0
