File: PCBs/EpaperDisplayPCB.kicad_sch (KiCad schematic)
At the start: 21 parts, among them J1 Conn_01x08, J2 Conn_01x12_FPC_0.5mm, Q1 AO3404A, U1 ePaper-2.1

Commit message: fuck you
Parts:
- removed J2: Conn_01x12_FPC_0.5mm, SparkFun-Connector:FPC_12_0.5MM, symbol SparkFun-Connector:Conn_01x12_FPC_0.5mm
- removed U1: ePaper-2.1, SparkFun-Display:ePaper-2.13, symbol SparkFun-Display:ePaper-2.1
- added FID1, FID2, FID3, FID4: Fiducial_0.5mm, SparkFun-Aesthetic:Fiducial_0.5mm_Mask1mm, symbol SparkFun-Aesthetic:Fiducial_0.5mm
- added J1: Conn_01x12_FPC_0.5mm, SparkFun-Connector:FPC_12_0.5MM, symbol SparkFun-Connector:Conn_01x12_FPC_0.5mm
- added U1: ePaper-2.66, SparkFun-Display:ePaper-2.66, symbol SparkFun-Display:ePaper-2.66
- renumbered J1 to J2
Connections:
- net +3.3V: now also J2.1 (Pin_1), J1.1 (Pin_1), U1.15 (VDDIO), U1.16 (VDD); no longer J2.7 (Pin_7)
- net D/~{C}: now also J2.4 (Pin_4), J1.4 (Pin_4), U1.11 (D/~{C}); no longer J2.6 (Pin_6)
- net GND: now also J1.8 (Pin_8), U1.17 (GND), U1.8 (BS)
- net SCLK: now also J2.6 (Pin_6), J1.6 (Pin_6), U1.13 (SCLK); no longer J2.4 (Pin_4)
- net SDIO: now also J2.7 (Pin_7), J1.7 (Pin_7), U1.14 (SDIO); no longer J2.5 (Pin_5)
- net ~{BUSY}: now also J1.2 (Pin_2), U1.9 (~{BUSY})
- net ~{CS}: now also J2.5 (Pin_5), J1.5 (Pin_5), U1.12 (~{CS}); no longer J2.3 (Pin_3)
- net ~{RST}: now also J2.3 (Pin_3), J1.3 (Pin_3), U1.10 (~{RST}); no longer J2.1 (Pin_1)
- net at C5.1, D2.A: now also U1.23 (VGL)
- net at C4.1, D3.C: now also U1.21 (VGH)
- net at C8.1: now also U1.20 (VDH)
- net at C7.1: now also U1.18 (VDDD)
- net at Q1.1 (G): now also U1.2 (GDR)
- net at C9.1: now also U1.22 (VDL)
- net at C10.1: now also U1.24 (VCOM)
- net at Q1.2 (S), R1.2: now also U1.3 (RESE)
- net at C6.1: now also U1.5 (VDHR)
- no-connect marks 0 -> 4
Other:
- note added: "Connectors"
- note added: "Fiducials"
- moved on the sheet: J2
