File: PCBs/EpaperDisplayPCB.kicad_sch (KiCad schematic)
At the start: 31 parts, among them J1 Conn_01x12_FPC_0.5mm, J2 Conn_01x08, Q1 AO3404A, U1 ePaper-2.66, U2 LIS3DH

Commit message: Adding Fiducials to Epaper
Adding stencil alignment fiducials to epaper PCB
Parts:
- added FID10, FID11, FID12, FID13, FID14, FID15, FID5, FID6, FID7, FID8, FID9: Fiducial_3mm, SparkFun-Aesthetic:Fiducial_1.5mm_Mask3mm, symbol SparkFun-Aesthetic:Fiducial_3mm
Other:
- note added: "Stencil Fiducials"
