File: PCBs/MainBoard.kicad_pcb (KiCad board)
At the start: 2 copper layers, 40.4 x 70 mm, 76 parts, among them J1 USB_C_Receptacle, J2 Conn_01x12_FPC_0.5mm, J3 Conn_01x08, J4 Qwiic_RA, SW1 PTH_RA_h7.5mm, SW2 SMD_4.6x2.8mm_h2.5mm, U1 TVS_ESD_USB, U2 ESP32-S3-MINI, U3 AP3012, U4 MQ-4 Gas Sensor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

Commit message: Adding updates From review
Fixed epaper to main board FPC connection.
Added fiducials to main board for stencil alignment purposes.
Parts:
- added FID10: Fiducial_3mm, SparkFun-Aesthetic:Fiducial_1.5mm_Mask3mm, F.Cu at (134.0, 133.1)
- added FID11: Fiducial_3mm, SparkFun-Aesthetic:Fiducial_1.5mm_Mask3mm, F.Cu at (164.0, 133.1)
- added FID12: Fiducial_3mm, SparkFun-Aesthetic:Fiducial_1.5mm_Mask3mm, F.Cu at (181.0, 118.9)
- added FID13: Fiducial_3mm, SparkFun-Aesthetic:Fiducial_1.5mm_Mask3mm, F.Cu at (181.0, 88.9)
- added FID14: Fiducial_3mm, SparkFun-Aesthetic:Fiducial_1.5mm_Mask3mm, F.Cu at (181.0, 58.9)
- added FID5: Fiducial_3mm, SparkFun-Aesthetic:Fiducial_1.5mm_Mask3mm, F.Cu at (134.0, 44.6)
- added FID6: Fiducial_3mm, SparkFun-Aesthetic:Fiducial_1.5mm_Mask3mm, F.Cu at (117.0, 58.9)
- added FID7: Fiducial_3mm, SparkFun-Aesthetic:Fiducial_1.5mm_Mask3mm, F.Cu at (117.0, 88.9)
- added FID8: Fiducial_3mm, SparkFun-Aesthetic:Fiducial_1.5mm_Mask3mm, F.Cu at (117.0, 118.9)
- added FID9: Fiducial_3mm, SparkFun-Aesthetic:Fiducial_1.5mm_Mask3mm, F.Cu at (164.0, 44.6)
Connections:
- J2 pad 1: +3.3V -> unconnected-(J2-Pin_1-Pad1)
- J2 pad 10: SDA -> ~{RST}
- J2 pad 11: unconnected-(J2-Pin_11-Pad11) -> ~{BUSY}
- J2 pad 12: unconnected-(J2-Pin_12-Pad12) -> +3.3V
- J2 pad 2: ~{BUSY} -> unconnected-(J2-Pin_2-Pad2)
- J2 pad 3: ~{RST} -> SDA
- J2 pad 4: D/~{C} -> SCL
- J2 pad 5: ~{CS} -> GND
- J2 pad 6: SCLK -> SDIO
- J2 pad 7: SDIO -> SCLK
- J2 pad 8: GND -> ~{CS}
- J2 pad 9: SCL -> D/~{C}
- J3 pad 2: ~{BUSY} -> SDIO
- J3 pad 3: ~{RST} -> SCLK
- J3 pad 4: D/~{C} -> ~{CS}
- J3 pad 5: ~{CS} -> D/~{C}
- J3 pad 6: SCLK -> ~{RST}
- J3 pad 7: SDIO -> ~{BUSY}
- U2 pad 34: ~{BUSY} -> SDIO
- U2 pad 35: ~{RST} -> SCLK
- U2 pad 36: D/~{C} -> ~{CS}
- U2 pad 37: ~{CS} -> D/~{C}
- U2 pad 38: SCLK -> ~{RST}
- U2 pad 39: SDIO -> ~{BUSY}
Routing:
- net ~{BUSY}: track 15.1 -> 20.1 mm, vias 0 -> 2
- net SDIO: track 21.3 -> 17.1 mm, vias 2 -> 0
- net SDA: track 64.6 -> 62.1 mm
- net GND: track 97.0 -> 99.2 mm, vias 42 -> 49
- net SCL: track 73.0 -> 71.1 mm
- net ~{RST}: track 13.8 -> 15.5 mm
- net D/~{C}: track 13.1 -> 14.5 mm
- net SCLK: track 14.7 -> 15.8 mm
- net ~{CS}: track 13.6 -> 14.4 mm
- net +3.3V: track 167.6 -> 167.1 mm
Other:
- board text added: "v13.5"
- board text removed: "v13.4"
