File: PCBs/MainBoard-ESP-MQ-Control.kicad_pcb (KiCad board)
At the start: 2 copper layers, 40.4 x 70 mm, 86 parts, among them J1 USB_C_Receptacle, J2 Conn_01x12_FPC_0.5mm, J3 Conn_01x08, J4 Qwiic_RA, SW1 PTH_RA_h7.5mm, SW2 SMD_4.6x2.8mm_h2.5mm, U1 TVS_ESD_USB, U2 ESP32-S3-MINI, U3 AP3012, U4 MQ-4 Gas Sensor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

Commit message: Edits
Making edits
Parts:
- added Q1: DMG2305UX, SparkFun-Semiconductor-Standard:SOT23-3, F.Cu at (152.3, 78.9)
- added Q2: DMG2305UX, SparkFun-Semiconductor-Standard:SOT23-3, F.Cu at (135.2, 66.1)
- moved R7 10.3 mm to (143.4, 90.2), turned to 0 degrees
Connections:
- U2 pad 21: unconnected-(U2-IOA17-Pad21) -> ~{SHDN}-EN
- U2 pad 22: ~{SHDN}-EN -> MQ7-CONTROL
- U2 pad 29: unconnected-(U2-IO34-Pad29) -> MQ4-CONTROL
- U4 pad 1: +5V -> MQ4-5V
- U4 pad 2: +5V -> MQ4-5V
- U4 pad 3: +5V -> MQ4-5V
- U7 pad 1: +5V -> MQ7-5V
- U7 pad 2: +5V -> MQ7-5V
- U7 pad 3: +5V -> MQ7-5V
Routing:
- net MQ4-CONTROL: track 0.00 -> 43.5 mm, vias 0 -> 2
- net MQ7-CONTROL: track 0.00 -> 23.6 mm
- net +5V: track 109.4 -> 91.4 mm
- net MQ4-5V: track 0.00 -> 17.2 mm, vias 0 -> 2
- net MQ7-5V: track 0.00 -> 15.1 mm
- net ESP11/MQ4: track 46.9 -> 50.9 mm
- net GND: track 99.2 -> 98.5 mm
